Commit message: almost clean and working build

File: src/p3dx/PioneerModel/p3dx_description/urdf/pioneer3dx_wheel.xacro (robot description, xacro)
@@ -87,5 +87,7 @@
     <transmission name="${parent}_${suffix}_wheel_trans">
       <type>pr2_mechanism_model/SimpleTransmission</type>
-      <joint name="base_${suffix}_wheel_joint" />
+      <joint name="base_${suffix}_wheel_joint">
+	<hardwareInterface>EffortJointInterface</hardwareInterface>
+      </joint>
       <actuator name="base_${suffix}_wheel_motor">
         <hardwareInterface>EffortJointInterface</hardwareInterface>
