Commit message: Solved null colliders bug and added all the launch scripts

File: src/p3dx/xacro/p3dx/pioneer3dx.xacro (robot description, xacro)
@@ -2,16 +2,16 @@
 <robot xmlns:xacro="http://www.ros.org/wiki/xacro" name="pioneer3dx" >
   <!-- Import Rviz colors -->
-  <xacro:include filename="$(find gazebo_plugins)/test/multi_robot_scenario/xacro/materials.xacro" />
+  <xacro:include filename="$(find p3dx)/xacro/materials.xacro" />
   <!-- Import robot -->
-  <xacro:include filename="$(find gazebo_plugins)/test/multi_robot_scenario/xacro/p3dx/pioneer3dx_body.xacro"/>
+  <xacro:include filename="$(find p3dx)/xacro/p3dx/pioneer3dx_body.xacro"/>
   <xacro:pioneer3dx_body name="chassis" parent="base_link" meshes="package://gazebo_plugins/test/multi_robot_scenario/meshes/p3dx"/>
   <!-- Laser  -->
-  <xacro:include filename="$(find gazebo_plugins)/test/multi_robot_scenario/xacro/laser/hokuyo.xacro"/>
+  <xacro:include filename="$(find p3dx)/xacro/laser/hokuyo.xacro"/>
   <xacro:laser name="front_laser" parent="chassis" xyz="0.16 0 0.1" rpy="0 0 0" meshes="package://gazebo_plugins/test/multi_robot_scenario/meshes/laser"/>
   <!-- GPU Laser
-  <xacro:include filename="$(find gazebo_plugins)/test/multi_robot_scenario/xacro/laser/hokuyo_gpu.xacro"/>
+  <xacro:include filename="$(find p3dx)/xacro/laser/hokuyo_gpu.xacro"/>
   <xacro:laser_gpu name="front_laser" parent="chassis" xyz="0.16 0 0.1" rpy="0 0 0" meshes="package://gazebo_plugins/test/multi_robot_scenario/meshes/laser" />
     -->
-  <xacro:include filename="$(find gazebo_plugins)/test/multi_robot_scenario/xacro/camera/camera.xacro"/>
+  <xacro:include filename="$(find p3dx)/xacro/camera/camera.xacro"/>
   <xacro:cam name="front_camera" parent="chassis" xyz="0 0 0.5" rpy="0 0 0" />
 </robot>

File: src/p3dx/xacro/p3dx/pioneer3dx_sonar.xacro (robot description, xacro)
@@ -27,5 +27,5 @@
       <origin xyz="0 0 0" rpy="0 0 0"/>
       <geometry>
-        <box size="0 0 0"/>
+        <box size="0.01 0.01 0.01"/>
       </geometry>
     </collision>

File: src/p3dx/xacro/p3dx/pioneer3dx_swivel.xacro (robot description, xacro)
@@ -31,5 +31,5 @@
       <origin xyz="0 0 0" rpy="0 0 0"/>
       <geometry>
-        <box size="0 0 0"/>
+        <box size="0.01 0.01 0.01"/>
       </geometry>
     </collision>
@@ -98,5 +98,5 @@
       <origin xyz="0 0 0" rpy="0 0 0"/>
       <geometry>
-        <box size="0 0 0"/>
+        <box size="0.01 0.01 0.01"/>
       </geometry>
     </collision>

File: src/p3dx/xacro/p3dx/pioneer3dx_wheel.xacro (robot description, xacro)
@@ -29,5 +29,5 @@
       <origin xyz="0 0 0" rpy="0 0 0"/>
       <geometry>
-        <box size="0 0 0"/>
+        <box size="0.01 0.01 0.01"/>
       </geometry>
     </collision>
